Commit message: to do code test

File: src/fmauch_universal_robot/ur_description/urdf/inc/ur_macro.xacro (robot description, xacro)
@@ -66,6 +66,6 @@
   <xacro:arg name="publish_pointcloud" default="false" />
   <xacro:include filename="$(find realsense_ros_gazebo)/xacro/depthcam.xacro"/>
-  <xacro:realsense_d435 sensor_name="d435" parent_link="wrist_3_link" rate="10">
-    <origin xyz="-0.1 0. 0.0" rpy="${pi} ${-pi/2} 0"/>
+  <xacro:realsense_d435 sensor_name="d435" parent_link="wrist_3_link" rate="10" publish_pointcloud="true">
+    <origin xyz="-0.1 0. 0.0" rpy="0 ${-pi/2} 0"/>
   </xacro:realsense_d435>
   <xacro:macro name="ur_robot" params="
